Commit message: Add UR Series

File: Robots/UR_Series/UR5/urdf/UR5.urdf (robot description, URDF)
Before this commit: robot UniversalRobots_UR5, 8 links, 7 joints
Links:
- link BaseLink: geometry collision mesh filename=package://UR5/Collision/BaseLink.stl; visual mesh filename=package://UR5/Visual/BaseLink.dae
- link Link1: geometry collision mesh filename=package://UR5/Collision/Link1.stl; visual mesh filename=package://UR5/Visual/Link1.dae
- link Link2: geometry collision mesh filename=package://UR5/Collision/Link2.stl; visual mesh filename=package://UR5/Visual/Link2.dae
- link Link3: geometry collision mesh filename=package://UR5/Collision/Link3.stl; visual mesh filename=package://UR5/Visual/Link3.dae
- link Link4: geometry collision mesh filename=package://UR5/Collision/Link4.stl; visual mesh filename=package://UR5/Visual/Link4.dae
- link Link5: geometry collision mesh filename=package://UR5/Collision/Link5.stl; visual mesh filename=package://UR5/Visual/Link5.dae
- link Link6: geometry collision mesh filename=package://UR5/Collision/Link6.stl; visual mesh filename=package://UR5/Visual/Link6.dae
